File: Moxie.kicad_pcb (KiCad board)
At the start: 4 copper layers, 0 parts

Commit message: routing
Parts:
- added A1: Arduino_Nano_v3.x, Module:Arduino_Nano, F.Cu at (170.6, 93.6)
- added C1: 100n, Capacitor_THT:C_Disc_D7.0mm_W2.5mm_P5.00mm, F.Cu at (175.8, 67.2)
- added C2: 100n, Capacitor_THT:C_Disc_D7.0mm_W2.5mm_P5.00mm, F.Cu at (176.0, 79.5)
- added C3: 100n, Capacitor_THT:C_Disc_D7.0mm_W2.5mm_P5.00mm, F.Cu at (175.9, 92.5)
- added D1: LED, LED_THT:LED_D5.0mm, F.Cu at (192.0, 55.5)
- added R1: 1k, Resistor_THT:R_Axial_DIN0207_L6.3mm_D2.5mm_P7.62mm_Horizontal, F.Cu at (181.8, 68.8)
- added R2: 1k, Resistor_THT:R_Axial_DIN0207_L6.3mm_D2.5mm_P7.62mm_Horizontal, F.Cu at (182.0, 80.8)
- added R3: 1k, Resistor_THT:R_Axial_DIN0207_L6.3mm_D2.5mm_P7.62mm_Horizontal, F.Cu at (181.9, 93.2)
- added R4: 1k, Resistor_THT:R_Axial_DIN0207_L6.3mm_D2.5mm_P7.62mm_Horizontal, F.Cu at (175.4, 55.0)
- added SW1: SW_Push, Button_Switch_THT:SW_PUSH_6mm, F.Cu at (187.6, 63.0)
- added SW2: SW_Push, Button_Switch_THT:SW_PUSH_6mm, F.Cu at (187.5, 75.0)
- added SW3: SW_Push, Button_Switch_THT:SW_PUSH_6mm, F.Cu at (187.4, 87.5)
- added U1: MAX30102, spo2:MAX30102_MODULE, F.Cu at (135.0, 90.0)
- added U2: SSD1306, spo2:SSD1306, F.Cu at (137.4, 66.5)
Routing:
- net +5V: track 0.00 -> 56.4 mm
- net Net-(A1-D4): track 0.00 -> 24.8 mm
- net Net-(A1-D3): track 0.00 -> 23.9 mm
- net Net-(A1-D2): track 0.00 -> 23.7 mm
- net Net-(D1-A): track 0.00 -> 6.65 mm
- net Net-(A1-D12): track 0.00 -> 6.02 mm
- added copper zone on B.Cu, net GND
- added copper zone on F.Cu, net GND
